File: hardware/OpenRX-Gemini.kicad_pcb (KiCad board)
At the start: 6 copper layers, 17 x 15.7 mm, 86 parts, among them J1 Conn_Coaxial_Small, J2 Conn_Coaxial_Small, T1 0900PC16J0042001E, T2 0900PC16J0042001E, U1 ESP32-C3, U2 TLV75533PDQNR, U3 LR1121IMLTRT, U4 RFX2401C, U5 SKY13373-460LF, U6 LR1121IMLTRT, U7 RFX2401C, U8 SKY13373-460LF, U9 TS2306A 240GF MSM 9_C2976675, X1 CJ17-400001010B20

Commit message: Rebrand OpenRX Gemini for DroneAid
Other:
- board text added: "DroneAid"
- board text removed: "OPEN"
